Commit message: controllers tested and joints with nicer names

File: robot_description/robot.urdf (robot description, URDF)
Before this commit: robot onshape, 4 links, 3 joints
Joints:
- removed joint 996_firstlink
- removed joint Revolute_firsttosecondlink
- removed joint Slider_actuator
- added joint joint1: type revolute, parent servomg996r, child first_link, origin xyz=6.505213034913026604e-18 0.0099999999999999915345 0.047499999999999993616 rpy=3.141592653589793116 2.4637214511932053286e-22 0.10904934252795142613, axis 0 0 1, limit effort=1 velocity=20
- added joint joint2: type revolute, parent first_link, child second_link, origin xyz=-0.00050000000000000304617 -0.059750000000000011435 -0.055999999999999987288 rpy=1.7662033618514959478e-21 2.5217203946365817101e-22 -5.465863304373380401e-15, axis 0 0 1, limit effort=1 velocity=20
- added joint slider_actuator: type prismatic, parent second_link, child actuator, origin xyz=0.018325999999999991602 -0.051833589599999993491 0.018598077114628464024 rpy=-3.141592653589793116 -5.1171304803077346007e-18 -1.5707963267948961139, axis 0 0 1, limit effort=1 velocity=20

File: scara_ws/src/scara_description/urdf/robot.urdf.xacro (robot description, xacro)
@@ -109,5 +109,5 @@
     <child link="servomg996r"/>
   </joint>
-  <joint name="996_firstlink" type="revolute">
+  <joint name="joint1" type="revolute">
     <origin xyz="0 0.01 0.0475" rpy="3.14159 0 0.109"/>
     <parent link="servomg996r"/>
@@ -116,5 +116,5 @@
     <limit lower="-3.14" upper="3.14" effort="1" velocity="20"/>
   </joint>
-  <joint name="Revolute_firsttosecondlink" type="revolute">
+  <joint name="joint2" type="revolute">
     <origin xyz="-0.0005 -0.0598 -0.056" rpy="0 0 0"/>
     <parent link="first_link"/>
@@ -123,5 +123,5 @@
     <limit lower="-3.14" upper="3.14" effort="1" velocity="20"/>
   </joint>
-  <joint name="Slider_actuator" type="prismatic">
+  <joint name="slider_actuator" type="prismatic">
     <origin xyz="0.0183 -0.0518 0.0186" rpy="3.14159 0 -1.5708"/>
     <parent link="second_link"/>

File: scara_ws/src/scara_description/urdf/scara_ros2_control.xacro (robot description, xacro)
@@ -6,5 +6,5 @@
             <plugin>gz_ros2_control/GazeboSimSystem</plugin>
         </hardware>
-        <joint name="996_firstlink">
+        <joint name="joint1">
             <command_interface name="position">
                 <param name="min">-${PI / 2}</param>
@@ -13,5 +13,5 @@
             <state_interface name="position"/>
         </joint>
-        <joint name="Revolute_firsttosecondlink">
+        <joint name="joint2">
             <command_interface name="position">
                 <param name="min">-${PI / 2}</param>
@@ -20,5 +20,5 @@
             <state_interface name="position"/>
         </joint>
-        <joint name="Slider_actuator">
+        <joint name="slider_actuator">
             <command_interface name="position">
                 <param name="min">0.0</param>
