Commit message: Launch file for rviz2 display

File: scara_ws/src/scara_description/urdf/robot.urdf.xacro (robot description, xacro)
@@ -1,11 +1,5 @@
 <?xml version="1.0"?>
 <robot xmlns:xacro="http://www.ros.org/wiki/xacro" name="scara">
-  <link name="base_link">
-    <inertial>
-      <origin xyz="0 0 0"/>
-      <mass value="0.1"/>
-      <inertia ixx="1e-5" ixy="0" ixz="0" iyy="1e-5" iyz="0" izz="1e-5"/>
-    </inertial>
-  </link>
+  <link name="base_link"/>
   <link name="servomg996r">
     <visual>

Commit message: Ros2_control xacro done for now

File: scara_ws/src/scara_description/urdf/robot.urdf.xacro (robot description, xacro)
@@ -3,5 +3,13 @@
   <xacro:arg name="is_ignition" default="true"/>
   <xacro:include filename="$(find scara_description)/urdf/scara_gazebo.xacro"/>
+  <xacro:include filename="$(find scara_description)/urdf/scara_ros2_control.xacro"/>
+  <!-- variables -->
+  <xacro:property name="PI" value="3.14159265359"/>
+  <xacro:property name="effort" value="30.0"/>
+  <xacro:property name="velocity" value="10.0"/>
   <link name="base_link"/>
+  <gazebo reference="base_link">
+    <static>true</static>
+  </gazebo>
   <link name="servomg996r">
     <visual>

Commit message: Configuration for controllers and some minor changes to the description and launch files

File: scara_ws/src/scara_description/urdf/robot.urdf.xacro (robot description, xacro)
@@ -8,8 +8,6 @@
   <xacro:property name="effort" value="30.0"/>
   <xacro:property name="velocity" value="10.0"/>
+  <link name="world"/>
   <link name="base_link"/>
-  <gazebo reference="base_link">
-    <static>true</static>
-  </gazebo>
   <link name="servomg996r">
     <visual>
@@ -101,4 +99,9 @@
   </link>
   <!-- Joints -->
+  <joint name="robot_in_world" type="fixed">
+    <origin xyz="0 0 0.0" rpy="0 0 0"/>
+    <parent link="world"/>
+    <child link="base_link"/>  <!-- or your robot's actual base link name -->
+  </joint>
   <joint name="base_to_servo" type="fixed">
     <origin xyz="0 0 0" rpy="0 0 0"/>

File: scara_ws/src/scara_description/urdf/scara_gazebo.xacro (robot description, xacro)
@@ -4,10 +4,10 @@
         <xacro:if value="$(arg is_ignition)">
             <plugin filename="ign_ros2_control-system" name="ign_ros2_control::IgnitionROS2ControlPlugin">
-                <parameters></parameters>
+                <parameters>$(find scara_controller)/config/scara_controllers.yaml</parameters>
             </plugin>
         </xacro:if>
         <xacro:unless value="$(arg is_ignition)">
-            <plugin filename="gz_ros2_control-system" name="gz_ros2_control::GazeboImROS2ControlPlugin">
-                <parameters></parameters>
+            <plugin filename="gz_ros2_control-system" name="gz_ros2_control::GazeboSimROS2ControlPlugin">
+                <parameters>$(find scara_controller)/config/scara_controllers.yaml</parameters>
             </plugin>
         </xacro:unless>

File: scara_ws/src/scara_description/urdf/scara_ros2_control.xacro (robot description, xacro)
@@ -33,5 +33,5 @@
             </command_interface>
             <state_interface name="position"/>
-            <state_interface name="velocity"/>
+<!--            <state_interface name="velocity"/>-->
         </joint>
     </ros2_control>

Commit message: Odeio tudo

File: scara_ws/src/scara_description/urdf/robot.urdf.xacro (robot description, xacro)
@@ -43,5 +43,5 @@
     </visual>
     <collision>
-      <origin xyz="0 0.01 0.0475" rpy="3.14159 0 0"/>
+      <origin xyz="0 0.01 0.047" rpy="3.14159 0 0"/>
       <geometry>
         <mesh filename="package://scara_description/meshes/first_link.stl"/>
@@ -65,5 +65,5 @@
     </visual>
     <collision>
-      <origin xyz="0.0005 0.07 0.1035" rpy="3.14159 0 0"/>
+      <origin xyz="0.0005 0.07 0.1025" rpy="3.14159 0 0"/>
       <geometry>
         <mesh filename="package://scara_description/meshes/second_link.stl"/>
@@ -87,7 +87,7 @@
     </visual>
     <collision>
-      <origin xyz="-0.1216 0.0178 -0.0916" rpy="0 0 -1.5708"/>
+      <origin xyz="0.0 -0.0178 0.04" rpy="0 0 -1.5708"/>
       <geometry>
-        <mesh filename="package://scara_description/meshes/actuator.stl"/>
+        <cylinder radius="0.005" length="0.12"/>
       </geometry>
     </collision>
@@ -102,5 +102,5 @@
     <origin xyz="0 0 0.0" rpy="0 0 0"/>
     <parent link="world"/>
-    <child link="base_link"/>  <!-- or your robot's actual base link name -->
+    <child link="base_link"/>
   </joint>
   <joint name="base_to_servo" type="fixed">

Commit message: Moveit planning working

File: scara_ws/src/scara_description/urdf/robot.urdf.xacro (robot description, xacro)
@@ -128,5 +128,5 @@
     <child link="actuator"/>
     <axis xyz="0 0 1"/>
-    <limit lower="0.0" upper="0.1" effort="1" velocity="0.2"/>
+    <limit lower="-0.1" upper="0.1" effort="1" velocity="0.2"/>
   </joint>
 </robot>

File: scara_ws/src/scara_description/urdf/scara_ros2_control.xacro (robot description, xacro)
@@ -26,4 +26,5 @@
             </command_interface>
             <state_interface name="position"/>
+            <param name="initial_position">0.0</param>
 <!--            <state_interface name="velocity"/>-->
         </joint>
